File: CatFeederUPS.kicad_pcb (KiCad board)
At the start: 2 copper layers, 75 x 22 mm, 19 parts, among them J1 JST-PH-2, J2 FEEDER-OUT, U2 BQ24079RGT, U3 TPS61235PRWLR

Commit message: pcb layout complete
Parts:
- moved R5 19.5 mm to (80.8, 59.8), turned to 180 degrees
- moved R8 19.2 mm to (80.8, 58.5), turned to 180 degrees
- moved R7 11.4 mm to (88.8, 59.5)
- moved C3 10.4 mm to (111.4, 56.6)
- moved C4 10.4 mm to (113.9, 56.6)
- moved C5 10.4 mm to (116.4, 56.6)
- moved D1 9.74 mm to (90.2, 64.7), turned to 0 degrees
- moved D2 9.34 mm to (90.3, 62.7)
- moved R4 8.28 mm to (87.9, 64.7), turned to 180 degrees
- moved R6 7.82 mm to (88.4, 62.2), turned to 90 degrees
Routing:
- net /VSYS: track 0.00 -> 45.6 mm, vias 0 -> 4
- net VIN: track 0.00 -> 40.1 mm, vias 0 -> 2
- net GND: track 0.00 -> 11.2 mm, vias 0 -> 13
- net VBAT: track 0.00 -> 10.6 mm
- net /VOUT: track 0.00 -> 4.36 mm
- net Net-(U2-~{PGOOD}): track 0.00 -> 3.63 mm
- net Net-(U3-SW): track 0.00 -> 3.61 mm
- net Net-(U2-ISET): track 0.00 -> 3.16 mm
- net Net-(U2-~{CHG}): track 0.00 -> 2.18 mm
- net Net-(U2-TS): track 0.00 -> 2.07 mm
- net Net-(U2-ILIM): track 0.00 -> 1.91 mm
- net Net-(D2-K): track 0.00 -> 1.36 mm
- net Net-(D1-K): track 0.00 -> 1.34 mm
- added copper zone on F.Cu, net /VOUT

Commit message: squish board
Parts:
- moved J1 20.3 mm to (79.8, 60.0)
- moved R5 9.24 mm to (90.1, 59.8)
- moved BT1 9.23 mm to (85.2, 62.1)
- moved C1 9.23 mm to (96.2, 57.5)
- moved C2 9.23 mm to (93.7, 63.5)
- moved C6 9.23 mm to (91.2, 63.0)
- moved D1 9.23 mm to (99.5, 64.7)
- moved D2 9.23 mm to (99.5, 62.7)
- moved R4 9.23 mm to (97.1, 64.7)
- moved R6 9.23 mm to (97.7, 62.2)
- moved R7 9.23 mm to (98.0, 59.5)
- moved R8 9.23 mm to (90.1, 58.5)
- moved U2 9.23 mm to (94.2, 60.5)
Routing:
- net VIN: track 40.1 -> 28.9 mm
- net /VSYS: track 45.6 -> 36.3 mm
- net GND: track 11.2 -> 12.9 mm
Other:
- board size 75 x 22 mm -> 49.4 x 11.2 mm

Commit message: throw some graphics on there
Parts:
- added G***: LOGO, ANT LOGO:antlogo, B.Cu at (102.8, 60.2)
Other:
- board text added: "Cat Feeder UPS"
- board text added: "Rev: ${REVISION}"

Commit message: fix LCSC part numbers, and the goddam TPS61235 footprint **again**
Parts:
- U3: footprint TPS61235P:RWL0009A -> ARGH:ARGH
Changed lines of the file:
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@@
 		(pcbplotparams
 			(layerselection 0x00000000_00000000_55555555_5755f5ff)
-			(plot_on_all_layers_selection 0x00000000_00000000_00000000_00000000)
+			(plot_on_all_layers_selection 0x00000000_00000000_00000000_0200a0af)
 			(disableapertmacros no)
-			(usegerberextensions no)
+			(usegerberextensions yes)
 			(usegerberattributes yes)
 			(usegerberadvancedattributes yes)
@@
 			(outputformat 1)
 			(mirror no)
-			(drillshape 1)
+			(drillshape 0)
 			(scaleselection 1)
-			(outputdirectory "")
+			(outputdirectory "gerbers/")
 		)
 	)
@@
 			)
 		)
+		(property "LCSC" "C140287"
+			(at 0 0 0)
+			(unlocked yes)
+			(layer "F.Fab")
+			(hide yes)
+			(effects
+				(font
+					(size 1 1)
+					(thickness 0.15)
+				)
+			)
+		)
 		(property ki_fp_filters "VQFN*1EP*3x3mm*P0.5mm*")
 		(sheetname "/")
@@
 			)
 		)
-		(property "LCSC" "C11702"
+		(property "LCSC" "C453521"
 			(at 0 0 180)
 			(unlocked yes)
@@
 			)
 		)
-		(property "LCSC" "C11702"
+		(property "LCSC" "C114759"
 			(at 0 0 180)
 			(unlocked yes)
@@
 			)
 		)
-		(attr through_hole)
+		(attr through_hole exclude_from_bom)
 		(duplicate_pad_numbers_are_jumpers no)
 		(fp_line
@@
 		)
 	)
-	(footprint "TPS61235P:RWL0009A"
+	(footprint "ARGH:ARGH"
 		(layer "F.Cu")
 		(at 110 60)
 		(tags "TPS61235PRWLR ")
 		(property "Reference" "U3"
-			(at 0 2.76 0)
+			(at 0 -2.54 0)
 			(unlocked yes)
 			(layer "F.SilkS")
-			(hide yes)
 			(effects
 				(font
@@
 		)
 		(property "Value" "TPS61235PRWLR"
-			(at 0 0 0)
+			(at 0 5.08 0)
 			(unlocked yes)
 			(layer "F.Fab")
-			(hide yes)
 			(effects
 				(font
@@
 			(fill yes)
 			(layer "F.Mask")
-			(net "Net-(U3-SW)")
 		)
 		(fp_line
@@
 		)
 		(fp_text user "${REFERENCE}"
-			(at 0 0 0)
+			(at 0 2.54 0)
 			(unlocked yes)
 			(layer "F.Fab")
@@
 			(pinfunction "PGND_1")
 			(pintype "power_in")
-			(zone_connect 2)
 		)
 		(pad "2" smd custom
@@
 			(pinfunction "VOUT_9")
 			(pintype "power_out")
-			(zone_connect 2)
 		)
 		(embedded_fonts no)
@@
 			)
 		)
-		(attr through_hole)
+		(attr through_hole exclude_from_bom)
 		(duplicate_pad_numbers_are_jumpers no)
 		(fp_line
@@
 			)
 		)
-		(property "LCSC" "C2286"
+		(property "LCSC" "C12624"
 			(at 0 0 0)
 			(unlocked yes)
@@
 			)
 		)
-		(property "LCSC" "C11702"
+		(property "LCSC" "C60490"
 			(at 0 0 180)
 			(unlocked yes)
@@
 			)
 		)
-		(property "LCSC" "C11702"
+		(property "LCSC" "C114759"
 			(at 0 0 90)
 			(unlocked yes)
@@
 			)
 		)
-		(property "LCSC" "C11702"
+		(property "LCSC" "C3016052"
 			(at 0 0 0)
 			(unlocked yes)
@@
 			)
 		)
-		(attr through_hole)
+		(attr through_hole exclude_from_bom)
 		(duplicate_pad_numbers_are_jumpers no)
 		(fp_line
@@
 			)
 		)
-		(property "LCSC" "C408536"
+		(property "LCSC" "C695604"
 			(at 0 0 0)
 			(unlocked yes)
@@
 		(effects
 			(font
-				(size 0.5 0.5)
+				(size 0.8 0.8)
 				(thickness 0.1)
 				(bold yes)

Commit message: a couple more component swaps, and away into production we go!
Routing:
- net GND: track 12.9 -> 11.4 mm
- net /VSYS: track 36.3 -> 35.4 mm
Changed lines of the file:
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@@
 			)
 		)
-		(property "LCSC" "C2286"
+		(property "LCSC" "C130719"
 			(at 0 0 0)
 			(unlocked yes)
@@
 			)
 		)
-		(property "LCSC" "C453521"
+		(property "LCSC" "C67014"
 			(at 0 0 180)
 			(unlocked yes)
@@
 			)
 		)
-		(property "Description" ""
+		(property "Description" "8-A valley current, 5.1-V fixed output voltage synchronous boost converters"
 			(at 0 0 0)
 			(layer "F.Fab")
@@
 		(sheetname "/")
 		(sheetfile "CatFeederUPS.kicad_sch")
+		(units
+			(unit
+				(name "A")
+				(pins "7" "6" "3" "4" "2" "9" "8" "5" "1")
+			)
+		)
 		(clearance 0.1)
 		(attr smd)
@@
 			)
 		)
-		(property "LCSC" "C12624"
+		(property "LCSC" "C74338"
 			(at 0 0 0)
 			(unlocked yes)
@@
 	)
 	(segment
-		(start 93.985 58.47)
-		(end 93.395 57.88)
-		(width 0.2)
-		(layer "F.Cu")
-		(net "GND")
-	)
-	(segment
 		(start 92.7975 61.25)
 		(end 92.255 61.7925)
@@
 		(net "GND")
 	)
-	(segment
-		(start 93.985 58.47)
-		(end 93.985 59.0625)
-		(width 0.2)
-		(layer "F.Cu")
-		(net "GND")
-	)
 	(via
 		(at 108.2 57.3)
@@
 	)
 	(segment
-		(start 97.675 60.86)
-		(end 98.285 60.25)
-		(width 0.2)
-		(layer "F.Cu")
-		(net "/VSYS")
-	)
-	(segment
 		(start 103.33 63.15)
 		(end 102.3 62.12)
@@
 	)
 	(segment
-		(start 97.205 60.86)
-		(end 97.675 60.86)
-		(width 0.2)
-		(layer "F.Cu")
-		(net "/VSYS")
-	)
-	(segment
 		(start 107.66 63.15)
 		(end 103.33 63.15)
@@
 	)
 	(via
-		(at 97.205 60.86)
+		(at 96.73 60.24)
 		(size 0.6)
 		(drill 0.3)
@@
 	)
 	(segment
+		(start 95.715 62.35)
+		(end 96.73 61.335)
+		(width 0.2)
+		(layer "B.Cu")
+		(net "/VSYS")
+	)
+	(segment
 		(start 95.485 65.03)
 		(end 95.715 64.8)
@@
 	)
 	(segment
-		(start 95.715 62.35)
-		(end 97.205 60.86)
+		(start 96.73 61.335)
+		(end 96.73 60.24)
 		(width 0.2)
 		(layer "B.Cu")
